File: dspod_h7r3/Hardware/dspod_h7r3.kicad_pcb (KiCad board)
At the start: 4 copper layers, 26.4 x 41.7 mm, 60 parts, among them J3 USB_C_Receptacle_USB2.0, J4 Conn_01x16, J5 Conn_01x16, P1 CONN_01X03, P5 CONN_01X06, SW1 SW_Push, SW2 SW_Push, U1 XC6222B331MR-G, U2 XC6222B331MR-G, U3 STM32H7R3V8Tx, U4 NAU88C22, U6 APS6404L-3SQR-SN, Y1 ABM10-167-12.000MHZ-T3

Commit message: Updated with minor tweaks for release to fab
Parts:
- added TP1: Diag0, TestPoint:TestPoint_Pad_D1.0mm, F.Cu at (143.9, 90.1)
- added TP2: Diag1, TestPoint:TestPoint_Pad_D1.0mm, F.Cu at (145.6, 88.8)
- added TP3: XSPI_NCS2, TestPoint:TestPoint_Pad_D1.0mm, B.Cu at (153.6, 93.5)
Connections:
- net /XSPI_NCS renamed /XSPI_NCS1
- U3 pad 29: unconnected-(U3-PD1-Pad29) -> /XSPI_NCS2
- U3 pad 71: unconnected-(U3-PC11-Pad71) -> Net-(U3-PC11)
- U3 pad 72: unconnected-(U3-PC12-Pad72) -> Net-(U3-PC12)
Routing:
- net /XSPI_NCS2: track 0.00 -> 14.8 mm, vias 0 -> 1
- net Net-(U3-PC11): track 0.00 -> 7.15 mm
- net Net-(U3-PC12): track 0.00 -> 5.63 mm
Other:
- board text added: "NCS2"
