File: dspod_h7r3/Hardware/dspod_h7r3.kicad_sch (KiCad schematic)
At the start: 60 parts, among them J3 USB_C_Receptacle_USB2.0, J4 Conn_01x16, J5 Conn_01x16, P1 CONN_01X03, P5 CONN_01X06, SW1 SW_Push, SW2 SW_Push, U1 XC6222B331MR-G, U2 XC6222B331MR-G, U3 STM32H7R3V8Tx, U4 NAU88C22, U6 APS6404L-3SQR-SN, Y1 ABM10-167-12.000MHZ-T3

Commit message: Updated with minor tweaks for release to fab
Parts:
- added TP1: Diag0, TestPoint:TestPoint_Pad_D1.0mm, symbol Connector:TestPoint
- added TP2: Diag1, TestPoint:TestPoint_Pad_D1.0mm, symbol Connector:TestPoint
- added TP3: XSPI_NCS2, TestPoint:TestPoint_Pad_D1.0mm, symbol Connector:TestPoint
Connections:
- net XSPI_NCS2: now reaches U3.29 (PO1)
- net XSPI_NCS2: now also TP3.1
- net at U3.71 (PC11): now also TP1.1
- net at U3.72 (PC12): now also TP2.1
- net XSPI_NCS renamed XSPI_NCS1
- no-connect marks 40 -> 37
Other:
- note added: "Alternate XSPI chip select for 2nd memory."
